File: iot1.sch (EAGLE design)
At the start: 53 parts, among them IC1 MEGA8-P, IC2 7805T, IC3 LTC2486C, IC4 7805T, IC5 4051N, IC6 OPA2134PA, J1 DCJ0202, U2 HTU21D, X1 22-23-2041, X2 A1944-50

Commit message: rearranging items
Connections:
- removed net N$43: IC1.PD2(INT0)
- removed net N$44: IC1.PD3(INT1)
- removed net N$45: IC1.PD4(XCK/T0)
- net MUX_0: now also IC1.PD2(INT0)
- net MUX_1: now also IC1.PD3(INT1)
- net MUX_2: now also IC1.PD4(XCK/T0)
Changed lines of the file:
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@@
 </segment>
 </net>
-<net name="N$43" class="0">
+<net name="MUX_0" class="0">
 <segment>
 <pinref part="IC1" gate="G$1" pin="PD2(INT0)"/>
 <wire x1="162.56" y1="137.16" x2="187.96" y2="137.16" width="0.1524" layer="91"/>
+<label x="190.5" y="137.16" size="1.778" layer="95"/>
 </segment>
 </net>
-<net name="N$44" class="0">
+<net name="MUX_1" class="0">
 <segment>
 <pinref part="IC1" gate="G$1" pin="PD3(INT1)"/>
 <wire x1="162.56" y1="134.62" x2="187.96" y2="134.62" width="0.1524" layer="91"/>
+<label x="190.5" y="134.62" size="1.778" layer="95"/>
 </segment>
 </net>
-<net name="N$45" class="0">
+<net name="MUX_2" class="0">
 <segment>
 <pinref part="IC1" gate="G$1" pin="PD4(XCK/T0)"/>
 <wire x1="162.56" y1="132.08" x2="187.96" y2="132.08" width="0.1524" layer="91"/>
+<label x="190.5" y="132.08" size="1.778" layer="95"/>
 </segment>
 </net>

Commit message: adding MAX485 module
Parts:
- added IC7: MAX3468CPA, maxim:MAX3468CPA
- added X3: 22-23-2041, con-molex:22-23-2041
Connections:
- new net N$43: X3-3.S
- new net N$44: X3-4.S
- new net N$7: X3-1.S
- new net N$8: X3-2.S
Other:
- note added: "Aquí se debería conectar el sensor que tiene una alimentación de 12V y 3 pines más que salen en la página de wsp"
- note added: "Este chip transforma de diferencial (salida del sensor de nuevo) a serial (hacia el arduino)"

Commit message: Step-up 5 to 12V
Parts:
- added C18: 0.1uF, rcl:C-EU025-024X044
- added C19: 0.33uF, rcl:C-EU025-024X044
- added C20: 680uF, rcl:C-EU025-024X044
- added D3: 1N5821, 1N5821:1N5821
- added L2: 100uH, rcl:L-EUL1812
- added R7: 2.2k, rcl:R-EU_0204/7
- added R8: 2k, rcl:R-EU_0204/7
- added R9: 17.4k, rcl:R-EU_0204/7
- added U3: LM2577T-ADJ/NOPB, LM2577T-ADJ_NOPB:LM2577T-ADJ/NOPB
Connections:
- new net 12V: C20.1, D3.K, R9.2
- new net N$45: D3.A, L2.2, U3.SWITCH
- new net N$84: R7.2, U3.COMP
- new net N$85: C19.1, R7.1
- new net N$87: R8.2, R9.1, U3.FEEDBACK
- net 5V: now also C18.1, L2.1, U3.VIN
- net GND: now also C18.2, C19.2, C20.2, R8.1, U3.GROUND
Changed lines of the file:
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@@
 <part name="X3" library="con-molex" library_urn="urn:adsk.eagle:library:165" deviceset="22-23-2041" device="" package3d_urn="urn:adsk.eagle:package:8078635/1"/>
 <part name="IC7" library="maxim" library_urn="urn:adsk.eagle:library:269" deviceset="MAX34*" device="PA" package3d_urn="urn:adsk.eagle:package:29519/2" technology="68C"/>
+<part name="FRAME7" library="frames" library_urn="urn:adsk.eagle:library:229" deviceset="A4L-LOC" device=""/>
+<part name="U3" library="LM2577T-ADJ_NOPB" deviceset="LM2577T-ADJ/NOPB" device=""/>
+<part name="C18" library="rcl" library_urn="urn:adsk.eagle:library:334" deviceset="C-EU" device="025-024X044" package3d_urn="urn:adsk.eagle:package:23630/1" value="0.1uF"/>
+<part name="C19" library="rcl" library_urn="urn:adsk.eagle:library:334" deviceset="C-EU" device="025-024X044" package3d_urn="urn:adsk.eagle:package:23630/1" value="0.33uF"/>
+<part name="C20" library="rcl" library_urn="urn:adsk.eagle:library:334" deviceset="C-EU" device="025-024X044" package3d_urn="urn:adsk.eagle:package:23630/1" value="680uF"/>
+<part name="R7" library="rcl" library_urn="urn:adsk.eagle:library:334" deviceset="R-EU_" device="0204/7" package3d_urn="urn:adsk.eagle:package:23498/2" value="2.2k"/>
+<part name="R8" library="rcl" library_urn="urn:adsk.eagle:library:334" deviceset="R-EU_" device="0204/7" package3d_urn="urn:adsk.eagle:package:23498/2" value="2k"/>
+<part name="R9" library="rcl" library_urn="urn:adsk.eagle:library:334" deviceset="R-EU_" device="0204/7" package3d_urn="urn:adsk.eagle:package:23498/2" value="17.4k"/>
+<part name="L2" library="rcl" library_urn="urn:adsk.eagle:library:334" deviceset="L-EU" device="L1812" package3d_urn="urn:adsk.eagle:package:23494/2" value="100uH"/>
+<part name="D3" library="1N5821" deviceset="1N5821" device=""/>
 </parts>
 <sheets>
@@
 </segment>
 </net>
+</nets>
+</sheet>
+<sheet>
+<plain>
+</plain>
+<instances>
+<instance part="FRAME7" gate="G$1" x="-15.24" y="-27.94" smashed="yes">
+<attribute name="DRAWING_NAME" x="201.93" y="-12.7" size="2.54" layer="94"/>
+<attribute name="LAST_DATE_TIME" x="201.93" y="-17.78" size="2.286" layer="94"/>
+<attribute name="SHEET" x="215.265" y="-22.86" size="2.54" layer="94"/>
+</instance>
+<instance part="U3" gate="G$1" x="96.52" y="83.82" smashed="yes">
+<attribute name="NAME" x="81.28" y="92.202" size="1.778" layer="95"/>
+<attribute name="VALUE" x="81.28" y="73.66" size="1.778" layer="96"/>
+</instance>
+<instance part="C18" gate="G$1" x="58.42" y="101.6" smashed="yes">
+<attribute name="NAME" x="59.944" y="101.981" size="1.778" layer="95"/>
+<attribute name="VALUE" x="59.944" y="96.901" size="1.778" layer="96"/>
+</instance>
+<instance part="C19" gate="G$1" x="68.58" y="60.96" smashed="yes">
+<attribute name="NAME" x="70.104" y="61.341" size="1.778" layer="95"/>
+<attribute name="VALUE" x="70.104" y="56.261" size="1.778" layer="96"/>
+</instance>
+<instance part="C20" gate="G$1" x="147.32" y="93.98" smashed="yes">
+<attribute name="NAME" x="148.844" y="94.361" size="1.778" layer="95"/>
+<attribute name="VALUE" x="148.844" y="89.281" size="1.778" layer="96"/>
+</instance>
+<instance part="R7" gate="G$1" x="68.58" y="71.12" smashed="yes" rot="R90">
+<attribute name="NAME" x="67.0814" y="67.31" size="1.778" layer="95" rot="R90"/>
+<attribute name="VALUE" x="71.882" y="67.31" size="1.778" layer="96" rot="R90"/>
+</instance>
+<instance part="R8" gate="G$1" x="137.16" y="78.74" smashed="yes" rot="R90">
+<attribute name="NAME" x="135.6614" y="74.93" size="1.778" layer="95" rot="R90"/>
+<attribute name="VALUE" x="140.462" y="74.93" size="1.778" layer="96" rot="R90"/>
+</instance>
+<instance part="R9" gate="G$1" x="137.16" y="99.06" smashed="yes" rot="R90">
+<attribute name="NAME" x="135.6614" y="95.25" size="1.778" layer="95" rot="R90"/>
+<attribute name="VALUE" x="140.462" y="95.25" size="1.778" layer="96" rot="R90"/>
+</instance>
+<instance part="L2" gate="G$1" x="96.52" y="109.22" smashed="yes" rot="R90">
+<attribute name="NAME" x="100.33" y="107.7214" size="1.778" layer="95" rot="R180"/>
+<attribute name="VALUE" x="100.33" y="112.522" size="1.778" layer="96" rot="R180"/>
+</instance>
+<instance part="D3" gate="G$1" x="121.92" y="109.22" smashed="yes">
+<attribute name="NAME" x="116.84" y="111.76" size="1.778" layer="95"/>
+<attribute name="VALUE" x="116.84" y="105.41" size="1.778" layer="96"/>
+</instance>
+</instances>
+<busses>
+</busses>
+<nets>
+<net name="GND" class="0">
+<segment>
+<pinref part="U3" gate="G$1" pin="GROUND"/>
+<wire x1="116.84" y1="78.74" x2="116.84" y2="71.12" width="0.1524" layer="91"/>
+<label x="114.3" y="68.58" size="1.778" layer="95"/>
+</segment>
+<segment>
+<pinref part="C18" gate="G$1" pin="2"/>
+<wire x1="58.42" y1="96.52" x2="58.42" y2="91.44" width="0.1524" layer="91"/>
+<label x="55.88" y="88.9" size="1.778" layer="95"/>
+</segment>
+<segment>
+<pinref part="C19" gate="G$1" pin="2"/>
+<wire x1="68.58" y1="55.88" x2="68.58" y2="50.8" width="0.1524" layer="91"/>
+<label x="66.04" y="48.26" size="1.778" layer="95"/>
+</segment>
+<segment>
+<pinref part="R8" gate="G$1" pin="1"/>
+<wire x1="137.16" y1="73.66" x2="137.16" y2="68.58" width="0.1524" layer="91"/>
+<label x="134.62" y="66.04" size="1.778" layer="95"/>
+</segment>
+<segment>
+<pinref part="C20" gate="G$1" pin="2"/>
+<wire x1="147.32" y1="88.9" x2="147.32" y2="81.28" width="0.1524" layer="91"/>
+<label x="144.78" y="78.74" size="1.778" layer="95"/>
+</segment>
+</net>
+<net name="N$45" class="0">
+<segment>
+<pinref part="L2" gate="G$1" pin="2"/>
+<pinref part="D3" gate="G$1" pin="A"/>
+<wire x1="101.6" y1="109.22" x2="116.84" y2="109.22" width="0.1524" layer="91"/>
+<pinref part="U3" gate="G$1" pin="SWITCH"/>
+<wire x1="116.84" y1="88.9" x2="116.84" y2="109.22" width="0.1524" layer="91"/>
+<junction x="116.84" y="109.22"/>
+</segment>
+</net>
+<net name="5V" class="0">
+<segment>
+<pinref part="U3" gate="G$1" pin="VIN"/>
+<pinref part="L2" gate="G$1" pin="1"/>
+<wire x1="76.2" y1="88.9" x2="76.2" y2="109.22" width="0.1524" layer="91"/>
+<wire x1="76.2" y1="109.22" x2="91.44" y2="109.22" width="0.1524" layer="91"/>
+<pinref part="C18" gate="G$1" pin="1"/>
+<wire x1="58.42" y1="104.14" x2="58.42" y2="109.22" width="0.1524" layer="91"/>
+<wire x1="58.42" y1="109.22" x2="76.2" y2="109.22" width="0.1524" layer="91"/>
+<junction x="76.2" y="109.22"/>
+<wire x1="58.42" y1="109.22" x2="50.8" y2="109.22" width="0.1524" layer="91"/>
+<junction x="58.42" y="109.22"/>
+<label x="45.72" y="109.22" size="1.778" layer="95"/>
+</segment>
+</net>
+<net name="N$84" class="0">
+<segment>
+<pinref part="U3" gate="G$1" pin="COMP"/>
+<wire x1="76.2" y1="83.82" x2="68.58" y2="83.82" width="0.1524" layer="91"/>
+<pinref part="R7" gate="G$1" pin="2"/>
+<wire x1="68.58" y1="83.82" x2="68.58" y2="76.2" width="0.1524" layer="91"/>
+</segment>
+</net>
+<net name="N$85" class="0">
+<segment>
+<pinref part="R7" gate="G$1" pin="1"/>
+<pinref part="C19" gate="G$1" pin="1"/>
+<wire x1="68.58" y1="66.04" x2="68.58" y2="63.5" width="0.1524" layer="91"/>
+</segment>
+</net>
+<net name="12V" class="0">
+<segment>
+<pinref part="D3" gate="G$1" pin="K"/>
+<pinref part="R9" gate="G$1" pin="2"/>
+<wire x1="127" y1="109.22" x2="137.16" y2="109.22" width="0.1524" layer="91"/>
+<wire x1="137.16" y1="109.22" x2="137.16" y2="104.14" width="0.1524" layer="91"/>
+<wire x1="137.16" y1="109.22" x2="147.32" y2="109.22" width="0.1524" layer="91"/>
+<junction x="137.16" y="109.22"/>
+<pinref part="C20" gate="G$1" pin="1"/>
+<wire x1="147.32" y1="109.22" x2="147.32" y2="96.52" width="0.1524" layer="91"/>
+<wire x1="147.32" y1="109.22" x2="154.94" y2="109.22" width="0.1524" layer="91"/>
+<junction x="147.32" y="109.22"/>
+<label x="157.48" y="109.22" size="1.778" layer="95"/>
+</segment>
+</net>
+<net name="N$87" class="0">
+<segment>
+<pinref part="R9" gate="G$1" pin="1"/>
+<pinref part="R8" gate="G$1" pin="2"/>
+<wire x1="137.16" y1="93.98" x2="137.16" y2="86.36" width="0.1524" layer="91"/>
+<pinref part="U3" gate="G$1" pin="FEEDBACK"/>
+<wire x1="137.16" y1="86.36" x2="137.16" y2="83.82" width="0.1524" layer="91"/>
+<wire x1="116.84" y1="86.36" x2="137.16" y2="86.36" width="0.1524" layer="91"/>
+<junction x="137.16" y="86.36"/>
+</segment>
+</net>

Commit message: Entrada Sensor de Temperatura y Humedad Ambiente
Parts:
- added X4: 22-23-2041, con-molex:22-23-2041
Connections:
- net 5V: now also X4-3.S
- net GND: now also X4-4.S
- net SCL: now also X4-2.S
- net SDA: now also X4-1.S
Changed lines of the file:
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@@
 <part name="L2" library="rcl" library_urn="urn:adsk.eagle:library:334" deviceset="L-EU" device="L1812" package3d_urn="urn:adsk.eagle:package:23494/2" value="100uH"/>
 <part name="D3" library="1N5821" deviceset="1N5821" device=""/>
+<part name="X4" library="con-molex" library_urn="urn:adsk.eagle:library:165" deviceset="22-23-2041" device="" package3d_urn="urn:adsk.eagle:package:8078635/1"/>
 </parts>
 <sheets>
@@
 <attribute name="VALUE" x="87.63" y="85.598" size="1.778" layer="96"/>
 </instance>
+<instance part="X4" gate="-1" x="119.38" y="30.48" smashed="yes">
+<attribute name="NAME" x="121.92" y="29.718" size="1.524" layer="95"/>
+<attribute name="VALUE" x="118.618" y="31.877" size="1.778" layer="96"/>
+</instance>
+<instance part="X4" gate="-2" x="119.38" y="27.94" smashed="yes">
+<attribute name="NAME" x="121.92" y="27.178" size="1.524" layer="95"/>
+</instance>
+<instance part="X4" gate="-3" x="119.38" y="25.4" smashed="yes">
+<attribute name="NAME" x="121.92" y="24.638" size="1.524" layer="95"/>
+</instance>
+<instance part="X4" gate="-4" x="119.38" y="22.86" smashed="yes">
+<attribute name="NAME" x="121.92" y="22.098" size="1.524" layer="95"/>
+</instance>
 </instances>
 <busses>
@@
 <label x="101.6" y="71.12" size="1.778" layer="95"/>
 </segment>
+<segment>
+<pinref part="X4" gate="-4" pin="S"/>
+<wire x1="116.84" y1="22.86" x2="104.14" y2="22.86" width="0.1524" layer="91"/>
+<label x="96.52" y="22.86" size="1.778" layer="95"/>
+</segment>
 </net>
 <net name="SOIL_MOISTURE_1" class="0">
@@
 <label x="78.74" y="109.22" size="1.778" layer="95"/>
 </segment>
+<segment>
+<pinref part="X4" gate="-3" pin="S"/>
+<wire x1="116.84" y1="25.4" x2="104.14" y2="25.4" width="0.1524" layer="91"/>
+<label x="96.52" y="25.4" size="1.778" layer="95"/>
+</segment>
 </net>
 <net name="SDA" class="0">
@@
 <label x="172.72" y="142.24" size="1.778" layer="95"/>
 </segment>
+<segment>
+<pinref part="X4" gate="-1" pin="S"/>
+<wire x1="116.84" y1="30.48" x2="104.14" y2="30.48" width="0.1524" layer="91"/>
+<label x="96.52" y="30.48" size="1.778" layer="95"/>
+</segment>
 </net>
 <net name="N$31" class="0">
@@
 <label x="172.72" y="139.7" size="1.778" layer="95"/>
 </segment>
-</net>
+<segment>
+<pinref part="X4" gate="-2" pin="S"/>
+<wire x1="116.84" y1="27.94" x2="104.14" y2="27.94" width="0.1524" layer="91"/>
+<label x="96.52" y="27.94" size="1.778" layer="95"/>
+</segment>
+</net>

Commit message: LED
Parts:
- added LED1: (no value), led:LED3MM
- added R10: 680, rcl:R-EU_0207/10
Connections:
- new net N$76: LED1.C, R10.2
- net GND: now also R10.1
- net N$15: now also LED1.A
Changed lines of the file:
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@@
 <part name="D3" library="1N5821" deviceset="1N5821" device=""/>
 <part name="X4" library="con-molex" library_urn="urn:adsk.eagle:library:165" deviceset="22-23-2041" device="" package3d_urn="urn:adsk.eagle:package:8078635/1"/>
+<part name="LED1" library="led" library_urn="urn:adsk.eagle:library:259" deviceset="LED" device="3MM" package3d_urn="urn:adsk.eagle:package:15797/1"/>
+<part name="R10" library="rcl" library_urn="urn:adsk.eagle:library:334" deviceset="R-EU_" device="0207/10" package3d_urn="urn:adsk.eagle:package:23491/2" value="680"/>
 </parts>
 <sheets>
@@
 <attribute name="VALUE" x="55.499" y="138.684" size="1.778" layer="96" rot="R90"/>
 </instance>
+<instance part="LED1" gate="G$1" x="200.66" y="175.26" smashed="yes" rot="R90">
+<attribute name="NAME" x="205.232" y="178.816" size="1.778" layer="95" rot="R180"/>
+<attribute name="VALUE" x="205.232" y="180.975" size="1.778" layer="96" rot="R180"/>
+</instance>
+<instance part="R10" gate="G$1" x="215.9" y="175.26" smashed="yes" rot="R180">
+<attribute name="NAME" x="219.71" y="173.7614" size="1.778" layer="95" rot="R180"/>
+<attribute name="VALUE" x="219.71" y="178.562" size="1.778" layer="96" rot="R180"/>
+</instance>
 </instances>
 <busses>
@@
 <segment>
 <pinref part="IC1" gate="G$1" pin="PC0(ADC0)"/>
-<wire x1="162.56" y1="165.1" x2="187.96" y2="165.1" width="0.1524" layer="91"/>
+<wire x1="162.56" y1="165.1" x2="190.5" y2="165.1" width="0.1524" layer="91"/>
+<wire x1="190.5" y1="165.1" x2="190.5" y2="175.26" width="0.1524" layer="91"/>
+<pinref part="LED1" gate="G$1" pin="A"/>
+<wire x1="190.5" y1="175.26" x2="198.12" y2="175.26" width="0.1524" layer="91"/>
 </segment>
 </net>
@@
 <label x="35.56" y="144.78" size="1.778" layer="95"/>
 </segment>
+<segment>
+<pinref part="R10" gate="G$1" pin="1"/>
+<wire x1="220.98" y1="175.26" x2="226.06" y2="175.26" width="0.1524" layer="91"/>
+<label x="228.6" y="175.26" size="1.778" layer="95"/>
+</segment>
 </net>
 <net name="5V" class="0">
@@
 </segment>
 </net>
+<net name="N$76" class="0">
+<segment>
+<pinref part="LED1" gate="G$1" pin="C"/>
+<pinref part="R10" gate="G$1" pin="2"/>
+<wire x1="205.74" y1="175.26" x2="210.82" y2="175.26" width="0.1524" layer="91"/>
+</segment>
+</net>

Commit message: adding MAX3468
Parts:
- removed D3: 1N5821, 1N5821:1N5821
- removed IC7: MAX3468CPA, maxim:MAX3468CPA
- removed X3: 22-23-2041, con-molex:22-23-2041
- added C21: (no value), rcl:C-EU025-024X044
- added D4, D5, D6, D7, D8: 1N4004, diode:1N4004
- added IC8: MAX3468CPA, maxim:MAX3468CPA
- added R11, R22, R23: (no value), rcl:R-EU_0207/10
- added X5: 22-23-2041, con-molex:22-23-2041
Connections:
- removed net N$23: IC1.PC3(ADC3)
- removed net N$43: X3-3.S
- removed net N$44: X3-4.S
- removed net N$7: X3-1.S
- removed net N$8: X3-2.S
- new net 485A: D6.C, D7.A, IC8.A, R11.1, R22.2, X5-3.S
- new net 485B: D4.A, D5.C, IC8.B, R11.2, R23.1, X5-4.S
- new net N$88: IC8.DI
- new net TX_485: IC1.PC3(ADC3), IC8.RO
- net 12V: now also D8.C, X5-1.S; no longer D3.K
- net 3.3V: now also C21.1, IC8.VCC, R22.1
- net 5V: now also D4.C, D7.C
- net GND: now also C21.2, D5.A, D6.A, IC8.DE, IC8.GND, IC8.RE/, R23.2, X5-2.S
- net N$45: now also D8.A; no longer D3.A
Other:
- note removed: "Aquí se debería conectar el sensor que tiene una alimentación de 12V y 3 pines más que salen en la página de wsp"
- note removed: "Este chip transforma de diferencial (salida del sensor de nuevo) a serial (hacia el arduino)"

Commit message: renumbering board components
Parts:
- removed D8: 1N4004, diode:1N4004
- removed IC8: MAX3468CPA, maxim:MAX3468CPA
- removed X5: 22-23-2041, con-molex:22-23-2041
- added D3: 1N4004, diode:1N4004
- added IC7: LTC2486C, linear-technology:LTC2486C
- added X3: 22-23-2041, con-molex:22-23-2041
- C10: value 0.1u -> 10u
- C11: value 1u -> (none); device rcl:C-EU050-025X075 -> rcl:C-EU025-024X044
- C12: value 10u -> (none)
- C13: value 0.1u -> (none); device rcl:C-EU050-025X075 -> rcl:C-EUC0603
- C14: value (none) -> 0.1u; device rcl:C-EUC0603 -> rcl:C-EU050-025X075
- C15, C16: device rcl:C-EUC0603 -> rcl:C-EU050-025X075
- C18: value 0.1uF -> (none); device rcl:C-EU025-024X044 -> rcl:C-EUC0603
- C19: value 0.33uF -> (none); device rcl:C-EU025-024X044 -> rcl:CPOL-EUE1.8-4
- C2: value (none) -> 0.1uF; device rcl:C-EU050-025X075 -> rcl:C-EU025-024X044
- C20: value 680uF -> (none); device rcl:C-EU025-024X044 -> rcl:CPOL-EUE1.8-4
- C21: device rcl:C-EU025-024X044 -> rcl:C-EUC0603
- C3: value (none) -> 1u
- C4: value (none) -> 0.33uF; device rcl:C-EU050-025X075 -> rcl:C-EU025-024X044
- C5, C6: device rcl:CPOL-EUE1.8-4 -> rcl:C-EU050-025X075
- C7: value (none) -> 680uF; device rcl:C-EU050-025X075 -> rcl:C-EU025-024X044
- C8: value (none) -> 0.1u
- IC1: value MEGA8-P -> OPA2134PA; device atmel:MEGA8-P -> linear:OPA2134PA
- IC2: value 7805T -> MEGA8-P; device linear:7805T -> atmel:MEGA8-P
- IC3: value LTC2486C -> 4051N; device linear-technology:LTC2486C -> 40xx:4051N
- IC5: value 4051N -> 7805T; device 40xx:4051N -> linear:7805T
- IC6: value OPA2134PA -> MAX3468CPA; device linear:OPA2134PA -> maxim:MAX3468CPA
- L1: value (none) -> 100uH; device rcl:L-US0207/7 -> rcl:L-EUL1812
- L2: value 100uH -> (none); device rcl:L-EUL1812 -> rcl:L-US0207/7
- R10: value 680 -> (none)
- R13: value (none) -> 10k; device rcl:R-EU_0207/10 -> rcl:R-EU_0204/5
- R16: value (none) -> 2k; device rcl:R-EU_0207/10 -> rcl:R-EU_0204/7
- R17: value (none) -> 17.4k; device rcl:R-EU_0207/10 -> rcl:R-EU_0204/7
- R20, R21: device rcl:R-EU_0207/10 -> rcl:R-EU_0204/7
- R3: value (none) -> 680; device rcl:R-EU_0204/7 -> rcl:R-EU_0207/10
- R4: value (none) -> 2.2k
- R5: value 10k -> (none); device rcl:R-EU_0204/5 -> rcl:R-EU_0207/10
- R7: value 2.2k -> (none); device rcl:R-EU_0204/7 -> rcl:R-EU_0207/10
- R8: value 2k -> (none); device rcl:R-EU_0204/7 -> rcl:R-EU_0207/10
- R9: value 17.4k -> (none); device rcl:R-EU_0204/7 -> rcl:R-EU_0207/10
- U1: value (none) -> HTU21D; device FaBo-LoRa:CMWX1ZZABZ -> SparkFun-Sensors:HTU21DSMD
- U2: value HTU21D -> LM2577T-ADJ/NOPB; device SparkFun-Sensors:HTU21DSMD -> LM2577T-ADJ_NOPB:LM2577T-ADJ/NOPB
- U3: value LM2577T-ADJ/NOPB -> (none); device LM2577T-ADJ_NOPB:LM2577T-ADJ/NOPB -> FaBo-LoRa:CMWX1ZZABZ
- X1: value 22-23-2041 -> A1944-50; device con-molex:22-23-2041 -> con-coax:A1944-50
- X2: value A1944-50 -> 22-23-2041; device con-coax:A1944-50 -> con-molex:22-23-2041
- renumbered STANDOFF2 to STANDOFF3
Connections:
- net 12V: now also C7.1, D1.C, R17.2, X2-1.S; no longer C20.1, D8.C, R9.2, X5-1.S
- net 3.3V: now also C11.1, C3.2, C8.2, IC5.VO, IC6.VCC, R19.1, U1.VDD, U3.VDD_MCU, U3.VDD_RF, U3.VREF+; no longer C11.2, C12.2, C21.1, IC4.VO, IC8.VCC, R22.1, U1.VDD_MCU, U1.VDD_RF, U1.VREF+, U2.VDD
- net 485A: now also D3.A, D4.C, IC6.A, R19.2, R22.1, X2-3.S; no longer D6.C, D7.A, IC8.A, R11.1, R22.2, X5-3.S
- net 485B: now also D2.A, IC6.B, R18.1, R22.2, X2-4.S; no longer D4.A, IC8.B, R11.2, R23.1, X5-4.S
- net 5V: now also C12.1, C13.1, C17.1, C19.+, D2.C, D3.C, D6.C, IC1A.V+, IC2.VCC@1, IC3P.VCC, IC4.VO, IC5.VI, IC7.VCC, IC7.VREF+, L1.1, R11.1, R20.2, R6.1, U2.VIN, X3-3.S; no longer C14.1, C15.1, C16.1, C6.+, D1.C, D4.C, D7.C, IC1.VCC@1, IC2.VO, IC3.VCC, IC3.VREF+, IC4.VI, IC5P.VCC, IC6A.V+, L2.1, R15.1, R17.1, R3.2, U3.VIN, X4-3.S
- net GND: now also C11.2, C12.2, C13.2, C14.1, C15.1, C16.1, C19.-, C20.-, C4.2, C5.1, C6.1, C7.2, D4.A, D7.A, IC1A.V-, IC2.GND@1, IC3A.INH, IC3P.GND, IC3P.VEE, IC5.GND, IC6.DE, IC6.GND, IC6.RE/, IC7.!CS, IC7.EXP, IC7.GND, IC7.VREF-, R13.1, R14.1, R15.1, R18.2, R3.1, U1.GND@2, U2.GROUND, U3.GND@25, U3.GND@27, U3.GND@44, U3.GND@49, U3.GND@50, U3.GND@51, U3.GND@52, U3.GND@53, U3.GND@54, U3.GND@55, U3.GND@56, U3.GND@57, U3.GND@7, X1.2, X2-2.S, X3-4.S, X4-2.S; no longer C11.1, C12.1, C13.1, C14.2, C15.2, C16.2, C19.2, C20.2, C4.1, C5.-, C6.-, C7.1, D2.A, D6.A, IC1.GND@1, IC2.GND, IC3.!CS, IC3.EXP, IC3.GND, IC3.VREF-, IC5A.INH, IC5P.GND, IC5P.VEE, IC6A.V-, IC8.DE, IC8.GND, IC8.RE/, R10.1, R21.1, R23.2, R5.1, R8.1, U1.GND@25, U1.GND@27, U1.GND@44, U1.GND@49, U1.GND@50, U1.GND@51, U1.GND@52, U1.GND@53, U1.GND@54, U1.GND@55, U1.GND@56, U1.GND@57, U2.GND@2, U2.GND@7, U3.GROUND, X1-2.S, X1-4.S, X2.2, X5-2.S
- net MUX_0: now also IC2.PD2(INT0), IC3A.A; no longer IC1.PD2(INT0), IC5A.A
- net MUX_1: now also IC2.PD3(INT1), IC3A.B; no longer IC1.PD3(INT1), IC5A.B
- net MUX_2: now also IC2.PD4(XCK/T0), IC3A.C; no longer IC1.PD4(XCK/T0), IC5A.C
- net N$1: now also U3.DBG_SX1276_DIO1; no longer U1.DBG_SX1276_DIO1
- net N$10: now also U3.GND@3; no longer U1.GND@3
- net N$11: now also U3.PA11; no longer U1.PA11
- net N$12: now also U3.PA12; no longer U1.PA12
- net N$13: now also R2.2; no longer R1.2
- net N$14: now also R1.2; no longer R2.2
- net N$15: now also IC2.PC0(ADC0); no longer IC1.PC0(ADC0)
- net N$16: now also IC2.PC1(ADC1); no longer IC1.PC1(ADC1)
- net N$17: now also U3.DBG_SX1276_DIO0; no longer U1.DBG_SX1276_DIO0
- net N$18: now also U3.PB15; no longer U1.PB15
- net N$19: now also U3.PB14; no longer U1.PB14
- net N$2: now also U3.DBG_SX1276_DIO5; no longer U1.DBG_SX1276_DIO5
- net N$20: now also U3.PB13; no longer U1.PB13
- net N$21: now also U3.PB12; no longer U1.PB12
- net N$22: now also IC2.PC2(ADC2); no longer IC1.PC2(ADC2)
- net N$24: now also U3.PA8; no longer U1.PA8
- net N$25: now also U3.PA5; no longer U1.PA5
- net N$26: now also U3.PA4; no longer U1.PA4
- net N$27: now also U3.PA3; no longer U1.PA3
- net N$28: now also U3.PA2; no longer U1.PA2
- net N$29: now also IC3A.X3; no longer IC5A.X3
- net N$3: now also U3.SX1276_DIO4; no longer U1.SX1276_DIO4
- net N$30: now also C6.2, L2.1, U3.ANT; no longer C8.2, L1.1, U1.ANT
- net N$31: now also IC7.SDO; no longer IC3.SDO
- net N$32: now also U3.DBG_CRF1; no longer U1.DBG_CRF1
- net N$33: now also U3.DBG_CRF3; no longer U1.DBG_CRF3
- net N$34: now also U3.DBG_CRF2; no longer U1.DBG_CRF2
- net N$35: now also U3.STSAFE_NRST; no longer U1.STSAFE_NRST
- net N$36: now also IC3A.X4; no longer IC5A.X4
- net N$37: now also U3.PA0; no longer U1.PA0
- net N$38: now also C14.2, U3.MCU_NRST; no longer C13.2, U1.MCU_NRST
- net N$39: now also U3.PB8; no longer U1.PB8
- net N$4: now also U3.DBG_SX1275_DIO3; no longer U1.DBG_SX1275_DIO3
- net N$40: now also U3.PB9; no longer U1.PB9
- net N$41: now also IC2.PD0(RXD); no longer IC1.PD0(RXD)
- net N$42: now also IC2.PD1(TXD); no longer IC1.PD1(TXD)
- net N$45: now also D1.A, L1.2, U2.SWITCH; no longer D8.A, L2.2, U3.SWITCH
- net N$46: now also U3.VDD_TCXO; no longer U1.VDD_TCXO
- net N$47: now also U3.TCXO_OUT; no longer U1.TCXO_OUT
- net N$48: now also U3.PH0-OSC_IN; no longer U1.PH0-OSC_IN
- net N$49: now also U3.PH1-OSC_OUT; no longer U1.PH1-OSC_OUT
- net N$5: now also U3.DBG_SX1276_DIO2; no longer U1.DBG_SX1276_DIO2
- net N$50: now also IC3A.X5; no longer IC5A.X5
- net N$51: now also R13.2, U3.BOOT0; no longer R5.2, U1.BOOT0
- net N$52: now also U3.SWCLK; no longer U1.SWCLK
- net N$53: now also U3.SWDIO; no longer U1.SWDIO
- net N$54: now also U3.PB5; no longer U1.PB5
- net N$55: now also U3.PB6; no longer U1.PB6
- net N$56: now also U3.PB7; no longer U1.PB7
- net N$57: now also U3.PB2; no longer U1.PB2
- net N$58: now also IC2.PD5(T1); no longer IC1.PD5(T1)
- net N$59: now also IC2.PD6(AIN0); no longer IC1.PD6(AIN0)
- net N$6: now also U3.VDD_USB; no longer U1.VDD_USB
- net N$60: now also IC2.PD7(AIN1); no longer IC1.PD7(AIN1)
- net N$61: now also IC2.PB0(ICP); no longer IC1.PB0(ICP)
- net N$62: now also IC2.PB1(OC1A); no longer IC1.PB1(OC1A)
- net N$63: now also IC2.PB2(SS/OC1B); no longer IC1.PB2(SS/OC1B)
- net N$64: now also IC2.PB3(MOSI/OC2); no longer IC1.PB3(MOSI/OC2)
- net N$65: now also IC3A.X6; no longer IC5A.X6
- net N$66: now also IC3A.X7; no longer IC5A.X7
- net N$67: now also IC2.PC6(/RESET), R20.1; no longer IC1.PC6(/RESET), R3.1
- net N$68: now also IC2.GND; no longer IC1.GND
- net N$69: now also IC2.AREF; no longer IC1.AREF
- net N$70: now also IC2.AVCC; no longer IC1.AVCC
- net N$71: now also IC7.CH3; no longer IC3.CH3
- net N$72: now also C15.2, IC2.PB7(XTAL2/TOSC2), R21.1; no longer C4.2, IC1.PB7(XTAL2/TOSC2), R4.1
- net N$73: now also C16.2, IC2.PB6(XTAL1/TOSC1), R21.2; no longer C3.2, IC1.PB6(XTAL1/TOSC1), R4.2
- net N$74: now also IC7.CH2; no longer IC3.CH2
- net N$75: now also IC7.CH1; no longer IC3.CH1
- net N$76: now also R3.2; no longer R10.2
- net N$77: now also IC7.COM; no longer IC3.COM
- net N$78: now also IC1A.+IN, R15.2, R5.1; no longer IC6A.+IN, R12.1, R16.2
- net N$81: now also IC1A.-IN, R9.2; no longer IC6A.-IN, R14.2
- net N$82: now also IC1B.+IN, R12.1, R14.2; no longer IC6B.+IN, R20.1, R21.2
- net N$83: now also IC1B.-IN, R8.2; no longer IC6B.-IN, R18.2
- net N$84: now also R4.2, U2.COMP; no longer R7.2, U3.COMP
- net N$85: now also C4.1, R4.1; no longer C19.1, R7.1
- net N$87: now also R16.2, R17.1, U2.FEEDBACK; no longer R8.2, R9.1, U3.FEEDBACK
- net N$88: now also IC6.DI; no longer IC8.DI
- net N$9: now also IC3A.X2; no longer IC5A.X2
- net RF_LORAWAN: now also C5.2, L2.2, X1.1; no longer C7.2, L1.2, X2.1
- net RX: now also IC2.PB4(MISO), U3.RX; no longer IC1.PB4(MISO), U1.RX
- net S: now also D6.A, D7.C, IC3A.X, R23.1; no longer D1.A, D2.C, IC5A.X, R6.1
- net SCL: now also IC2.PC5(ADC5/SCL), IC7.FO, IC7.SCK, R1.1, U1.SCK, X3-2.S; no longer IC1.PC5(ADC5/SCL), IC3.FO, IC3.SCK, R2.1, U2.SCK, X4-2.S
- net SDA: now also IC2.PC4(ADC4/SDA), IC7.SDI, R2.1, U1.DATA, X3-1.S; no longer IC1.PC4(ADC4/SDA), IC3.SDI, R1.1, U2.DATA, X4-1.S
- net SENSORS: now also C21.1, IC7.CH0, R23.2; no longer C17.1, IC3.CH0, R6.2
- net SOIL_MOISTURE_0: now also R11.2, R7.1, R9.1, X4-1.S; no longer R13.1, R14.1, R15.2, X1-1.S
- net SOIL_MOISTURE_1: now also R10.1, R6.2, R8.1, X4-3.S; no longer R17.2, R18.1, R19.1, X1-3.S
- net SOIL_MOISTURE_AMPLIFIED_0: now also IC1A.OUT, IC3A.X0, R5.2, R7.2; no longer IC5A.X0, IC6A.OUT, R12.2, R13.2
- net SOIL_MOISTURE_AMPLIFIED_1: now also IC1B.OUT, IC3A.X1, R10.2, R12.2; no longer IC5A.X1, IC6B.OUT, R19.2, R20.2
- net TX: now also IC2.PB5(SCK), U3.TX; no longer IC1.PB5(SCK), U1.TX
- net TX_485: now also IC2.PC3(ADC3), IC6.RO; no longer IC1.PC3(ADC3), IC8.RO
- net V_IN: now also C20.+, IC4.VI; no longer C5.+, IC2.VI
