File: iot1.sch (EAGLE design)
At the start: 75 parts, among them IC1 OPA2134PA, IC2 MEGA8-P, IC3 4051N, IC4 7805T, IC5 7805T, IC6 MAX3468CPA, IC7 LTC2486C, J1 DCJ0202, U1 HTU21D, U2 LM2577T-ADJ/NOPB, X1 A1944-50, X2 22-23-2041, X3 22-23-2041, X4 22-23-2041

Commit message: adding component's values
Parts:
- C11, C19: value (none) -> 0.1uF
- C12, C13, C15, C16: value (none) -> 100nF
- C17: value (none) -> 0.1pF
- C18: value (none) -> 10pF
- C20: value (none) -> 0.22uF
- C21: value (none) -> 1uF
- Q1: value (none) -> 16MHz
- R10, R11, R12, R14, R15, R5, R6, R7, R8, R9: value (none) -> 220
- R18, R19: value (none) -> 360
- R20: value (none) -> 10k
- R21, R23: value (none) -> 1M
- R22: value (none) -> 120
